File: DualSignalKontroll/untitled.kicad_sch (KiCad schematic)
At the start: 15 parts, among them J10 Buttons and switches, J11 Power Out, SW2 Switch B, SW3 Switch A, SW4 Switch A, SW5 Switch B, SW6 Select A, SW7 Select B

Commit message: initial code
Parts:
- removed J10 (x3): Buttons and switches, symbol Connector:Screw_Terminal_01x10
- removed J11 (x2): Power Out, symbol Connector:Screw_Terminal_01x03
- removed P1, P2, P3, P4: ~, symbol Connector:TestPoint
- removed SW2, SW5: Switch B, symbol Switch:SW_SPDT
- removed SW3, SW4: Switch A, symbol Switch:SW_SPDT
- removed SW6: Select A, symbol Switch:SW_Push
- removed SW7: Select B, symbol Switch:SW_Push
Other:
- note removed: "Alt. 1"
- note removed: "Alt. 2"
- note removed: "Antar at disse bruker boardets 12V power Da skal intern Gnd koples til"
- note removed: "Antar at disse bruker egen 10V/12V power Da skal ikke boardes 10V anvendes, men Gnd koples til"
- note removed: "Closed Thrown"
