File: DualSignalKontroll/DualSignalKontroll.kicad_sch (KiCad schematic)
At the start: 61 parts, among them J6 Signal A, J7 Signal B, J9 Power out, Q1 BC547, Q2 BC547, Q3 BC547, Q4 BC547, Q5 BC547, Q6 BC547, Q7 BD139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

Commit message: working with more debug info
Parts:
- removed JP5: Direct Conn TrackDetector, symbol Jumper:Jumper_3_Bridged12
Connections:
- net at U2.4: no longer A1.17 (D2)
- net at C1.1, R1.2: now also A1.17 (D2)
Other:
- note added: "A"
- note added: "B"
- note added: "C"
- note added: "D"
Changed lines of the file:
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@@
 		)
 	)
+	(text "B"
+		(exclude_from_sim no)
+		(at 189.738 93.218 0)
+		(effects
+			(font
+				(size 1.27 1.27)
+			)
+		)
+	)
 	(text "+12V"
 		(exclude_from_sim no)
@@
 		)
 	)
+	(text "D"
+		(exclude_from_sim no)
+		(at 189.992 95.758 0)
+		(effects
+			(font
+				(size 1.27 1.27)
+			)
+		)
+	)
 	(text "Red"
 		(exclude_from_sim no)
@@
 		)
 	)
+	(text "C"
+		(exclude_from_sim no)
+		(at 158.242 88.392 0)
+		(effects
+			(font
+				(size 1.27 1.27)
+			)
+		)
+	)
 	(text "Wires to 2nd board"
 		(exclude_from_sim no)
@@
 		)
 	)
+	(text "A"
+		(exclude_from_sim no)
+		(at 158.242 85.598 0)
+		(effects
+			(font
+				(size 1.27 1.27)
+			)
+		)
+	)
 	(text "Green 2"
 		(exclude_from_sim no)
@@
 	)
 	(junction
-		(at 109.22 78.74)
-		(diameter 0)
-		(color 0 0 0 0)
-	)
-	(junction
 		(at 71.12 121.92)
 		(diameter 0)
@@
 	(wire
 		(pts
+			(xy 83.82 63.5) (xy 83.82 69.85)
+		)
+		(stroke
+			(width 0)
+			(type default)
+		)
+	)
+	(wire
+		(pts
+			(xy 83.82 63.5) (xy 109.22 63.5)
+		)
+		(stroke
+			(width 0)
+			(type default)
+		)
+	)
+	(wire
+		(pts
 			(xy 121.92 140.97) (xy 265.43 140.97)
 		)
@@
 	(wire
 		(pts
-			(xy 102.87 78.74) (xy 109.22 78.74)
-		)
-		(stroke
-			(width 0)
-			(type default)
-		)
-	)
-	(wire
-		(pts
 			(xy 137.16 96.52) (xy 137.16 124.46)
 		)
@@
 	(wire
 		(pts
-			(xy 87.63 63.5) (xy 109.22 63.5)
-		)
-		(stroke
-			(width 0)
-			(type default)
-		)
-	)
-	(wire
-		(pts
 			(xy 46.99 78.74) (xy 57.15 78.74)
 		)
@@
 					(unit 1)
 				)
-			)
-		)
-	)
-	(symbol
-		(lib_id "Jumper:Jumper_3_Bridged12")
-		(at 87.63 69.85 270)
-		(mirror x)
-		(unit 1)
-		(exclude_from_sim no)
-		(in_bom no)
-		(on_board yes)
-		(dnp no)
-		(property "Reference" "JP5"
-			(at 90.17 68.5799 90)
-			(effects
-				(font
-					(size 1.27 1.27)
-				)
-				(justify left)
-			)
-		)
-		(property "Value" "Direct Conn TrackDetector"
-			(at 90.17 71.1199 90)
-			(effects
-				(font
-					(size 1.27 1.27)
-				)
-				(justify left)
-			)
-		)
-		(property "Footprint" ""
-			(at 87.63 69.85 0)
-			(effects
-				(font
-					(size 1.27 1.27)
-				)
-				(hide yes)
-			)
-		)
-		(property "Datasheet" "~"
-			(at 87.63 69.85 0)
-			(effects
-				(font
-					(size 1.27 1.27)
-				)
-				(hide yes)
-			)
-		)
-		(property "Description" "Jumper, 3-pole, pins 1+2 closed/bridged"
-			(at 87.63 69.85 0)
-			(effects
-				(font
-					(size 1.27 1.27)
-				)
-				(hide yes)
-			)
-		)
-		(pin "2"
-		)
-		(pin "3"
-		)
-		(pin "1"
-		)
-		(instances
-			(project ""
-				(path "/f90bb1a2-1a22-420b-b2f2-f9513faf4f93"
-					(reference "JP5")
-					(unit 1)
-				)
